Commit message: Lab2

File: Lab2/urdf/dynamic.urdf (robot description, URDF)
Before this commit: robot test_robot, 7 links, 6 joints
Links:
- removed link link3
- link arm1: geometry visual cylinder length=2 radius=0.05
- link arm2: geometry visual cylinder length=1 radius=0.05
- link arm3: geometry visual cylinder length=3 radius=0.025
- link base_link: geometry visual sphere radius=0.3
- link link1: geometry visual sphere radius=0.15
- link link2: geometry visual sphere radius=0.15
Joints:
- removed joint link3_to_arm3
- joint joint1: axis 0 0 1 -> 1 0 0; limit (none) -> lower=-3.14 upper=3.14 effort=1000.0 velocity=0.5; origin xyz=0 0 0 rpy=0 -0 0 -> xyz=0 0 0 rpy=0 1.57 0; type continuous -> revolute
- joint joint2: origin xyz=2 0 0 rpy=0 0 0 -> xyz=0 0 2 rpy=0 -1.57 0
- joint joint3: child link3 -> arm3; limit lower=0.3 upper=3 effort=1000.0 velocity=0.5 -> lower=0 upper=3 effort=1000.0 velocity=0.5

File: Lab2/urdf/static.urdf (robot description, URDF)
Before this commit: robot test_robot, 7 links, 6 joints
Links:
- removed link link3
- link arm1: geometry visual cylinder length=2 radius=0.05
- link arm2: geometry visual cylinder length=1 radius=0.05
- link arm3: geometry visual cylinder length=3 radius=0.025
- link base_link: geometry visual sphere radius=0.3
- link link1: geometry visual sphere radius=0.15
- link link2: geometry visual sphere radius=0.15
Joints:
- removed joint link3_to_arm3
- joint joint1: origin xyz=1 1.73025 0 rpy=0 -0 1.0472 -> xyz=0 0 0 rpy=0 1.57 0
- joint joint2: origin xyz=0.92388 0.382683 0 rpy=3.14159 -0 0.392699 -> xyz=0 0 2 rpy=0 -1.57 0
- joint joint3: child link3 -> arm3; origin xyz=0 0 2 rpy=0 0 0 -> xyz=1 0 0 rpy=3.14159 0 0
